File: grooveboard-choc-rp/grooveboard-choc-rp.kicad_pcb (KiCad board)
At the start: 2 copper layers, 120 x 25 mm, 47 parts, among them J1 USB_C_Receptacle_USB2.0, K1 MX-NoLED, K2 MX-NoLED, K3 MX-NoLED, K4 MX-NoLED, SW1 BOOT, SW2 RESET, U1 RP2040, U2 W25Q128JV, U3 AP2112K-3.3, Y1 12MHz

Commit message: update usb resistors
Other:
- board text added: "Grooveboard Choc RP v2.0"
- board text removed: "Grooveboard Choc RP v2.0 PROTO"
Changed lines of the file:
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@@
   (gr_arc (start 22.5 42.5) (end 20 42.5) (angle -90) (layer Edge.Cuts) (width 0.05))
   (gr_arc (start 22.5 22.5) (end 22.5 20) (angle -90) (layer Edge.Cuts) (width 0.05))
-  (gr_text "Grooveboard Choc RP v2.0 PROTO" (at 118.05 43.7) (layer B.SilkS)
+  (gr_text "Grooveboard Choc RP v2.0" (at 118.05 43.7) (layer B.SilkS)
     (effects (font (size 1 1) (thickness 0.15)) (justify mirror))
   )
